File: kicad/mag60lp_v1right/mag60lp_v1right.kicad_pcb (KiCad board)
At the start: 2 copper layers, 70 parts, among them U1 Arduino_Pro_Micro, U2 TRRS

Commit message: worked on cpb, but im  still so confused
Parts:
- D1, D10, D11, D12, D13, D14, D15, D16, D17, D18, D19, D2, D20, D21, D22, D23, D24, D25, D26, D27, D28, D29, D3, D30, D31, D32, D33, D34, D4, D5, D6, D7, D8, D9: moved to F.Cu
- S1, S10, S11, S12, S13, S14, S15, S16, S17, S18, S19, S2, S20, S22, S23, S24, S25, S26, S3, S4, S5, S6, S7, S8, S9: footprint ScottoKeebs_Choc:Choc_V1V2_1.00u -> ScottoKeebs_Choc:Choc_V2_1.00u
- S21: footprint ScottoKeebs_Choc:Choc_V1V2_2.00u -> ScottoKeebs_Choc:Choc_V2_2.00u
- S27, S29: footprint ScottoKeebs_Choc:Choc_V1V2_2.75u -> ScottoKeebs_Choc:Choc_V2_2.75u
- S28: footprint ScottoKeebs_Choc:Choc_V1V2_1.50u -> ScottoKeebs_Choc:Choc_V2_1.50u
- S30, S31, S32, S33: footprint ScottoKeebs_Choc:Choc_V1V2_1.25u -> ScottoKeebs_Choc:Choc_V2_1.25u
- S34: footprint ScottoKeebs_Choc:Choc_V1V2_2.25u -> ScottoKeebs_Choc:Choc_V2_2.25u
- moved U2 230.0 mm to (277.6, 82.8)
- moved U1 196.6 mm to (264.5, 98.6), turned to 0 degrees
- moved D15 185.8 mm to (267.4, 46.5), turned to 0 degrees
- moved D1 182.7 mm to (256.6, 39.4), turned to 0 degrees
- moved D29 182.7 mm to (278.1, 53.6), turned to 0 degrees
- moved D22 175.0 mm to (267.4, 71.3), turned to 0 degrees
- moved D8 172.6 mm to (256.6, 64.2), turned to 0 degrees
- moved D16 167.7 mm to (267.4, 50.0), turned to 0 degrees
- moved D2 164.4 mm to (256.6, 43.0), turned to 0 degrees
- moved D23 156.8 mm to (267.4, 74.9), turned to 0 degrees
- moved D9 154.3 mm to (256.6, 67.8), turned to 0 degrees
- moved D17 149.3 mm to (267.4, 53.6), turned to 0 degrees
- moved D30 149.3 mm to (278.1, 57.1), turned to 0 degrees
- moved D25 147.8 mm to (278.1, 39.4), turned to 0 degrees
- moved D3 146.1 mm to (256.6, 46.5), turned to 0 degrees
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Routing:
- net Column 4: track 252.5 -> 0.00 mm
- net Column 5: track 242.3 -> 0.00 mm
- net Column 6: track 240.1 -> 0.00 mm
- net Column 3: track 223.8 -> 0.00 mm
- net Column 2: track 214.9 -> 0.00 mm
- net Row 4: track 188.2 -> 0.00 mm, vias 2 -> 0
- net Row 2: track 187.7 -> 0.00 mm, vias 2 -> 0
- net Row 0: track 183.8 -> 0.00 mm
- net Row 3: track 173.0 -> 0.00 mm, vias 2 -> 0
- net Row 1: track 148.1 -> 0.00 mm
- net Column 0: track 105.7 -> 0.00 mm, vias 2 -> 0
- net Column 1: track 104.9 -> 0.00 mm
- net Net-(U1-RX1/PD2): track 100.7 -> 0.00 mm, vias 1 -> 0
- net Net-(U1-TX0/PD3): track 95.2 -> 0.00 mm
- net Net-(U2-RING2): track 76.3 -> 0.00 mm, vias 2 -> 0
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
Commit message: halfway through pcb
Parts:
- D1, D10, D11, D12, D13, D14, D15, D16, D17, D18, D19, D2, D20, D21, D22, D23, D24, D25, D26, D27, D28, D29, D3, D30, D31, D32, D33, D34, D4, D5, D6, D7, D8, D9: moved to B.Cu
- moved U2 228.6 mm to (54.1, 34.9)
- moved U1 195.1 mm to (69.5, 102.4), turned to 180 degrees
- moved D15 179.2 mm to (91.6, 81.2), turned to 90 degrees
- moved D1 178.6 mm to (78.1, 45.2), turned to 90 degrees
- moved D29 173.9 mm to (116.3, 117.3), turned to 90 degrees
- moved D8 169.5 mm to (87.1, 63.2), turned to 90 degrees
- moved D22 169.1 mm to (100.6, 99.2), turned to 90 degrees
- moved D16 160.8 mm to (109.6, 81.2), turned to 90 degrees
- moved D2 160.5 mm to (96.1, 45.2), turned to 90 degrees
- moved D9 151.6 mm to (105.1, 63.2), turned to 90 degrees
- moved D23 150.7 mm to (118.6, 99.2), turned to 90 degrees
- moved D3 142.5 mm to (114.1, 45.2), turned to 90 degrees
- moved D17 142.5 mm to (127.6, 81.2), turned to 90 degrees
- moved D30 139.4 mm to (152.3, 117.3), turned to 90 degrees
- moved D25 137.2 mm to (154.6, 99.2), turned to 90 degrees
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Routing:
- net Row 2: track 0.00 -> 140.2 mm
- net Row 1: track 0.00 -> 109.4 mm
- net Row 0: track 0.00 -> 109.3 mm

Commit message: pcb done?
i cant rember rn, i did this last night
Parts:
- added D35: Diode, ScottoKeebs_Components:Diode_DO-35, F.Cu at (78.9, 87.4)
- added SW1: SW_Push, Button_Switch_THT:SW_PUSH_6mm_H4.3mm, B.Cu at (74.8, 115.0)
- added SW2: SW_Push, Button_Switch_THT:SW_PUSH_6mm_H4.3mm, F.Cu at (64.8, 80.7)
- moved D27 26.5 mm to (180.9, 91.6), turned to 0 degrees
- moved D33 17.3 mm to (208.2, 104.4), turned to 0 degrees
- moved D21 12.7 mm to (201.5, 50.4), turned to 0 degrees
- moved D28 12.7 mm to (206.0, 68.4), turned to 0 degrees
- moved U1 3.46 mm to (72.6, 103.9)
- moved U2 2.50 mm to (55.6, 32.9)
- moved D34 0.08 mm to (210.9, 81.3)
Connections:
- U1 pad 22: unconnected-(U1-RST-Pad22) -> Net-(U1-RST)
- U1 pad 3: unconnected-(U1-GND-Pad3) -> Net-(SW1-Pad1)
Routing:
- net Column 4: track 0.00 -> 219.9 mm, vias 0 -> 9
- net Column 6: track 0.00 -> 215.6 mm, vias 0 -> 14
- net Column 5: track 0.00 -> 200.0 mm, vias 0 -> 14
- net Column 3: track 0.00 -> 199.4 mm, vias 0 -> 8
- net Row 4: track 0.00 -> 178.3 mm
- net Column 2: track 0.00 -> 159.1 mm, vias 0 -> 4
- net Row 3: track 0.00 -> 146.5 mm, vias 0 -> 2
- net Column 1: track 0.00 -> 138.1 mm, vias 0 -> 3
- net Column 0: track 0.00 -> 105.9 mm
- net Net-(U1-TX0/PD3): track 0.00 -> 89.0 mm
- net Net-(U2-RING2): track 0.00 -> 82.2 mm
- net Net-(U1-RX1/PD2): track 0.00 -> 81.5 mm
- net Net-(U1-VCC): track 0.00 -> 71.0 mm
- net Row 0: track 109.3 -> 175.6 mm
- net Row 1: track 109.4 -> 158.0 mm
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
Commit message: im losing my mind working on this
Parts:
- added J1: OLED_128x64, ScottoKeebs_Components:OLED_128x64, F.Cu at (58.8, 53.9)
- added J2: OLED_128x32, ScottoKeebs_Components:OLED_128x32, F.Cu at (162.5, 127.1)
- S1, S10, S11, S12, S13, S14, S15, S16, S17, S18, S19, S2, S20, S22, S23, S24, S25, S26, S3, S4, S5, S6, S7, S8, S9: footprint ScottoKeebs_Choc:Choc_V2_1.00u -> ScottoKeebs_Choc:Choc_V1V2_1.00u
- S21: footprint ScottoKeebs_Choc:Choc_V2_2.00u -> ScottoKeebs_Choc:Choc_V1V2_2.00u
- S27, S29: footprint ScottoKeebs_Choc:Choc_V2_2.75u -> ScottoKeebs_Choc:Choc_V1V2_2.75u
- S28: footprint ScottoKeebs_Choc:Choc_V2_1.50u -> ScottoKeebs_Choc:Choc_V1V2_1.50u
- S30, S31, S32, S33: footprint ScottoKeebs_Choc:Choc_V2_1.25u -> ScottoKeebs_Choc:Choc_V1V2_1.25u
- S34: footprint ScottoKeebs_Choc:Choc_V2_2.25u -> ScottoKeebs_Choc:Choc_V1V2_1.25u
- moved SW2 103.4 mm to (145.1, 145.9), turned to 0 degrees
- moved D35 85.5 mm to (144.7, 142.1), turned to 0 degrees
- moved U1 35.8 mm to (58.0, 71.3)
- moved SW1 27.3 mm to (58.9, 137.2)
Routing:
- net Column 4: track 219.9 -> 0.00 mm, vias 9 -> 0
- net Column 6: track 215.6 -> 0.00 mm, vias 14 -> 0
- net Column 5: track 200.0 -> 0.00 mm, vias 14 -> 0
- net Column 3: track 199.4 -> 0.00 mm, vias 8 -> 0
- net Row 4: track 178.3 -> 0.00 mm
- net Row 0: track 175.6 -> 0.00 mm
- net Column 2: track 159.1 -> 0.00 mm, vias 4 -> 0
- net Row 1: track 158.0 -> 0.00 mm
- net Row 3: track 146.5 -> 0.00 mm, vias 2 -> 0
- net Column 1: track 138.1 -> 0.00 mm, vias 3 -> 0
- net Row 2: track 120.5 -> 0.00 mm, vias 2 -> 0
- net Column 0: track 105.9 -> 0.00 mm
- net Net-(J1-SCL): track 89.0 -> 0.00 mm
- net Net-(J1-GND): track 82.2 -> 0.00 mm
- net Net-(J1-SDA): track 81.5 -> 0.00 mm
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