File: kicad/mag60lp_v1right/mag60lp_v1right.kicad_sch (KiCad schematic)
At the start: 70 parts, among them U1 Arduino_Pro_Micro, U2 TRRS

Commit message: worked on cpb, but im  still so confused
Parts:
- S1, S10, S11, S12, S13, S14, S15, S16, S17, S18, S19, S2, S20, S22, S23, S24, S25, S26, S3, S4, S5, S6, S7, S8, S9: footprint ScottoKeebs_Choc:Choc_V1V2_1.00u -> ScottoKeebs_Choc:Choc_V2_1.00u
- S21: footprint ScottoKeebs_Choc:Choc_V1V2_2.00u -> ScottoKeebs_Choc:Choc_V2_2.00u
- S27, S29: footprint ScottoKeebs_Choc:Choc_V1V2_2.75u -> ScottoKeebs_Choc:Choc_V2_2.75u
- S28: footprint ScottoKeebs_Choc:Choc_V1V2_1.50u -> ScottoKeebs_Choc:Choc_V2_1.50u
- S30, S31, S32, S33: footprint ScottoKeebs_Choc:Choc_V1V2_1.25u -> ScottoKeebs_Choc:Choc_V2_1.25u
- S34: footprint ScottoKeebs_Choc:Choc_V1V2_2.25u -> ScottoKeebs_Choc:Choc_V2_2.25u
Changed lines of the file:
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@@
 			)
 		)
-		(property "Footprint" "ScottoKeebs_Choc:Choc_V1V2_1.00u"
+		(property "Footprint" "ScottoKeebs_Choc:Choc_V2_1.00u"
 			(at 96.52 83.82 0)
 			(effects
@@
 			)
 		)
-		(property "Footprint" "ScottoKeebs_Choc:Choc_V1V2_1.00u"
+		(property "Footprint" "ScottoKeebs_Choc:Choc_V2_1.00u"
 			(at 76.2 101.6 0)
 			(effects
@@
 			)
 		)
-		(property "Footprint" "ScottoKeebs_Choc:Choc_V1V2_1.00u"
+		(property "Footprint" "ScottoKeebs_Choc:Choc_V2_1.00u"
 			(at 96.52 48.26 0)
 			(effects
@@
 			)
 		)
-		(property "Footprint" "ScottoKeebs_Choc:Choc_V1V2_1.00u"
+		(property "Footprint" "ScottoKeebs_Choc:Choc_V2_1.00u"
 			(at 96.52 66.04 0)
 			(effects
@@
 			)
 		)
-		(property "Footprint" "ScottoKeebs_Choc:Choc_V1V2_1.00u"
+		(property "Footprint" "ScottoKeebs_Choc:Choc_V2_1.00u"
 			(at 86.36 83.82 0)
 			(effects
@@
 			)
 		)
-		(property "Footprint" "ScottoKeebs_Choc:Choc_V1V2_1.00u"
+		(property "Footprint" "ScottoKeebs_Choc:Choc_V2_1.00u"
 			(at 96.52 101.6 0)
 			(effects
@@
 			)
 		)
-		(property "Footprint" "ScottoKeebs_Choc:Choc_V1V2_2.75u"
+		(property "Footprint" "ScottoKeebs_Choc:Choc_V2_2.75u"
 			(at 106.68 101.6 0)
 			(effects
@@
 			)
 		)
-		(property "Footprint" "ScottoKeebs_Choc:Choc_V1V2_1.25u"
+		(property "Footprint" "ScottoKeebs_Choc:Choc_V2_1.25u"
 			(at 86.36 119.38 0)
 			(effects
@@
 			)
 		)
-		(property "Footprint" "ScottoKeebs_Choc:Choc_V1V2_2.00u"
+		(property "Footprint" "ScottoKeebs_Choc:Choc_V2_2.00u"
 			(at 116.84 83.82 0)
 			(effects
@@
 			)
 		)
-		(property "Footprint" "ScottoKeebs_Choc:Choc_V1V2_1.00u"
+		(property "Footprint" "ScottoKeebs_Choc:Choc_V2_1.00u"
 			(at 66.04 66.04 0)
 			(effects
@@
 			)
 		)
-		(property "Footprint" "ScottoKeebs_Choc:Choc_V1V2_1.00u"
+		(property "Footprint" "ScottoKeebs_Choc:Choc_V2_1.00u"
 			(at 55.88 83.82 0)
 			(effects
@@
 			)
 		)
-		(property "Footprint" "ScottoKeebs_Choc:Choc_V1V2_1.00u"
+		(property "Footprint" "ScottoKeebs_Choc:Choc_V2_1.00u"
 			(at 55.88 66.04 0)
 			(effects
@@
 			)
 		)
-		(property "Footprint" "ScottoKeebs_Choc:Choc_V1V2_1.00u"
+		(property "Footprint" "ScottoKeebs_Choc:Choc_V2_1.00u"
 			(at 106.68 66.04 0)
 			(effects
@@
 			)
 		)
-		(property "Footprint" "ScottoKeebs_Choc:Choc_V1V2_1.00u"
+		(property "Footprint" "ScottoKeebs_Choc:Choc_V2_1.00u"
 			(at 106.68 83.82 0)
 			(effects
@@
 			)
 		)
-		(property "Footprint" "ScottoKeebs_Choc:Choc_V1V2_1.25u"
+		(property "Footprint" "ScottoKeebs_Choc:Choc_V2_1.25u"
 			(at 96.52 119.38 0)
 			(effects
@@
 			)
 		)
-		(property "Footprint" "ScottoKeebs_Choc:Choc_V1V2_2.25u"
+		(property "Footprint" "ScottoKeebs_Choc:Choc_V2_2.25u"
 			(at 106.68 119.38 0)
 			(effects
@@
 			)
 		)
-		(property "Footprint" "ScottoKeebs_Choc:Choc_V1V2_1.00u"
+		(property "Footprint" "ScottoKeebs_Choc:Choc_V2_1.00u"
 			(at 86.36 66.04 0)
 			(effects
@@
 			)
 		)
-		(property "Footprint" "ScottoKeebs_Choc:Choc_V1V2_1.00u"
+		(property "Footprint" "ScottoKeebs_Choc:Choc_V2_1.00u"
 			(at 66.04 83.82 0)
 			(effects
@@
 			)
 		)
-		(property "Footprint" "ScottoKeebs_Choc:Choc_V1V2_1.00u"
+		(property "Footprint" "ScottoKeebs_Choc:Choc_V2_1.00u"
 			(at 86.36 48.26 0)
 			(effects
@@
 			)
 		)
-		(property "Footprint" "ScottoKeebs_Choc:Choc_V1V2_1.00u"
+		(property "Footprint" "ScottoKeebs_Choc:Choc_V2_1.00u"
 			(at 55.88 48.26 0)
 			(effects
@@
 			)
 		)
-		(property "Footprint" "ScottoKeebs_Choc:Choc_V1V2_1.25u"
+		(property "Footprint" "ScottoKeebs_Choc:Choc_V2_1.25u"
 			(at 66.04 119.38 0)
 			(effects
@@
 			)
 		)
-		(property "Footprint" "ScottoKeebs_Choc:Choc_V1V2_1.00u"
+		(property "Footprint" "ScottoKeebs_Choc:Choc_V2_1.00u"
 			(at 116.84 48.26 0)
 			(effects
@@
 			)
 		)
-		(property "Footprint" "ScottoKeebs_Choc:Choc_V1V2_1.00u"
+		(property "Footprint" "ScottoKeebs_Choc:Choc_V2_1.00u"
 			(at 76.2 83.82 0)
 			(effects
@@
 			)
 		)
-		(property "Footprint" "ScottoKeebs_Choc:Choc_V1V2_1.00u"
+		(property "Footprint" "ScottoKeebs_Choc:Choc_V2_1.00u"
 			(at 86.36 101.6 0)
 			(effects
@@
 			)
 		)
-		(property "Footprint" "ScottoKeebs_Choc:Choc_V1V2_1.00u"
+		(property "Footprint" "ScottoKeebs_Choc:Choc_V2_1.00u"
 			(at 66.04 48.26 0)
 			(effects
@@
 			)
 		)
-		(property "Footprint" "ScottoKeebs_Choc:Choc_V1V2_1.25u"
+		(property "Footprint" "ScottoKeebs_Choc:Choc_V2_1.25u"
 			(at 76.2 119.38 0)
 			(effects
@@
 			)
 		)
-		(property "Footprint" "ScottoKeebs_Choc:Choc_V1V2_1.00u"
+		(property "Footprint" "ScottoKeebs_Choc:Choc_V2_1.00u"
 			(at 76.2 66.04 0)
 			(effects
@@
 			)
 		)
-		(property "Footprint" "ScottoKeebs_Choc:Choc_V1V2_1.00u"
+		(property "Footprint" "ScottoKeebs_Choc:Choc_V2_1.00u"
 			(at 116.84 66.04 0)
 			(effects
@@
 			)
 		)
-		(property "Footprint" "ScottoKeebs_Choc:Choc_V1V2_1.00u"
+		(property "Footprint" "ScottoKeebs_Choc:Choc_V2_1.00u"
 			(at 106.68 48.26 0)
 			(effects
@@
 			)
 		)
-		(property "Footprint" "ScottoKeebs_Choc:Choc_V1V2_2.75u"
+		(property "Footprint" "ScottoKeebs_Choc:Choc_V2_2.75u"
 			(at 55.88 119.38 0)
 			(effects
@@
 			)
 		)
-		(property "Footprint" "ScottoKeebs_Choc:Choc_V1V2_1.00u"
+		(property "Footprint" "ScottoKeebs_Choc:Choc_V2_1.00u"
 			(at 55.88 101.6 0)
 			(effects
@@
 			)
 		)
-		(property "Footprint" "ScottoKeebs_Choc:Choc_V1V2_1.00u"
+		(property "Footprint" "ScottoKeebs_Choc:Choc_V2_1.00u"
 			(at 66.04 101.6 0)
 			(effects
@@
 			)
 		)
-		(property "Footprint" "ScottoKeebs_Choc:Choc_V1V2_1.50u"
+		(property "Footprint" "ScottoKeebs_Choc:Choc_V2_1.50u"
 			(at 116.84 101.6 0)
 			(effects
@@
 			)
 		)
-		(property "Footprint" "ScottoKeebs_Choc:Choc_V1V2_1.00u"
+		(property "Footprint" "ScottoKeebs_Choc:Choc_V2_1.00u"
 			(at 76.2 48.26 0)
 			(effects

Commit message: pcb done?
i cant rember rn, i did this last night
Parts:
- added D35: Diode, ScottoKeebs_Components:Diode_DO-35, symbol ScottoKeebs:Placeholder_Diode
- added SW1, SW2: SW_Push, Button_Switch_THT:SW_PUSH_6mm_H4.3mm, symbol Switch:SW_Push
Connections:
- net Column 6: now also SW2.1
- net Row 4: now also D35.1 (K)
- net at U1.22 (RST): now also SW1.2
- net at U1.3 (GND): now also SW1.1
- new net: D35.2 (A), SW2.2

Commit message: im losing my mind working on this
Parts:
- added J1: OLED_128x64, ScottoKeebs_Components:OLED_128x64, symbol ScottoKeebs:OLED_128x64
- added J2: OLED_128x32, ScottoKeebs_Components:OLED_128x32, symbol ScottoKeebs:OLED_128x32
- S1, S10, S11, S12, S13, S14, S15, S16, S17, S18, S19, S2, S20, S22, S23, S24, S25, S26, S3, S4, S5, S6, S7, S8, S9: footprint ScottoKeebs_Choc:Choc_V2_1.00u -> ScottoKeebs_Choc:Choc_V1V2_1.00u
- S21: footprint ScottoKeebs_Choc:Choc_V2_2.00u -> ScottoKeebs_Choc:Choc_V1V2_2.00u
- S27, S29: footprint ScottoKeebs_Choc:Choc_V2_2.75u -> ScottoKeebs_Choc:Choc_V1V2_2.75u
- S28: footprint ScottoKeebs_Choc:Choc_V2_1.50u -> ScottoKeebs_Choc:Choc_V1V2_1.50u
- S30, S31, S32, S33: footprint ScottoKeebs_Choc:Choc_V2_1.25u -> ScottoKeebs_Choc:Choc_V1V2_1.25u
- S34: footprint ScottoKeebs_Choc:Choc_V2_2.25u -> ScottoKeebs_Choc:Choc_V1V2_1.25u
Connections:
- net at U1.1 (TX0/PD3), U2.3 (RING1): now also J1.3 (SCL)
- net at U1.2 (RX1/PD2), U2.2 (TIP): now also J1.4 (SDA)
- net at U1.21 (VCC), U2.1 (SLEEVE): now also J1.2 (VCC)
- net at U1.23 (GND), U2.4 (RING2): now also J1.1 (GND)
